Commit message: changed farmbot_urdf to farmbot_desctiption

File: farm_ws/src/farmbot_description/urdf/farmbot_description.urdf (robot description, URDF)
Before this commit: robot farmbot_urdf, 5 links, 4 joints
Links:
- link base_link: geometry collision mesh filename=package://farmbot_description/meshes/base_link.STL; visual mesh filename=package://farmbot_description/meshes/base_link.STL
- link front_wheel_left: geometry collision mesh filename=package://farmbot_description/meshes/front_wheel_left.STL; visual mesh filename=package://farmbot_description/meshes/front_wheel_left.STL
- link front_wheel_right: mass 75.2974306084417 -> 75.2974306084418; geometry collision mesh filename=package://farmbot_description/meshes/front_wheel_right.STL; visual mesh filename=package://farmbot_description/meshes/front_wheel_right.STL
- link rear_wheel_left: geometry collision mesh filename=package://farmbot_description/meshes/rear_wheel_left.STL; visual mesh filename=package://farmbot_description/meshes/rear_wheel_left.STL
- link rear_wheel_right: geometry collision mesh filename=package://farmbot_description/meshes/rear_wheel_right.STL; visual mesh filename=package://farmbot_description/meshes/rear_wheel_right.STL
Joints:
- joint front_wheel_left_joint: origin xyz=1.1332 1.1 -0.50637 rpy=0 0 0 -> xyz=1.13324967562402 1.1 -0.50636922357741 rpy=0 0 0
- joint front_wheel_right_joint: origin xyz=1.1332 -1.1 -0.50637 rpy=0 0 0 -> xyz=1.13324967562402 -1.1 -0.50636922357741 rpy=0 0 0
- joint rear_wheel_left_joint: origin xyz=-1.192 1.1 -0.50579 rpy=0 0 0 -> xyz=-1.19201296872286 1.1 -0.50579231398166 rpy=0 0 0
- joint rear_wheel_right_joint: origin xyz=-1.1937 -1.1 -0.50637 rpy=0 0 0 -> xyz=-1.1936883604935 -1.1 -0.50636922357741 rpy=0 0 0
